File: powermgr/powermgmt.sch (KiCad schematic (older format))
At the start: 3 parts, among them IC1 74HC4094_RevA_23Aug2012, J1 CONN_01X06, J2 CONN_01X06

Commit message: fixups and text
Parts:
- added C13: 100n, Capacitors_SMD:C_0805_HandSoldering, symbol CAP
- IC1: value 74HC4094_RevA_23Aug2012 -> CD4094
- J1: value CONN_01X06 -> IN; footprint Pin_Headers:Pin_Header_Angled_1x06_Pitch2.54mm -> Pin_Headers:Pin_Header_Straight_1x06_Pitch2.54mm
- J2: value CONN_01X06 -> OUT; footprint Pin_Headers:Pin_Header_Angled_1x06_Pitch2.54mm -> Pin_Headers:Pin_Header_Straight_1x06_Pitch2.54mm
Changed lines of the file:
@@
 P 1800 1600
 F 0 "IC1" H 1800 2050 50  0000 C CNN
-F 1 "74HC4094_RevA_23Aug2012" H 1800 1150 50  0000 C CNN
+F 1 "CD4094" H 1800 1150 50  0000 C CNN
 F 2 "Housings_SSOP:TSSOP-16_4.4x5mm_Pitch0.65mm" H 1800 1600 50  0001 C CNN
 F 3 "" H 1800 1600 50  0000 C CNN
@@
 ctrl_out0
 $Sheet
-S 3800 2000 1250 900
+S 3600 2750 1250 900
 U 5908DC66
 F0 "Power out" 60
@@
 P 2650 900
 F 0 "J2" H 2650 1250 50  0000 C CNN
-F 1 "CONN_01X06" V 2750 900 50  0000 C CNN
-F 2 "Pin_Headers:Pin_Header_Angled_1x06_Pitch2.54mm" H 2650 900 50  0001 C CNN
+F 1 "OUT" V 2750 900 50  0000 C CNN
+F 2 "Pin_Headers:Pin_Header_Straight_1x06_Pitch2.54mm" H 2650 900 50  0001 C CNN
 F 3 "" H 2650 900 50  0001 C CNN
 	1    2650 900
@@
 P 700 900
 F 0 "J1" H 700 1250 50  0000 C CNN
-F 1 "CONN_01X06" V 800 900 50  0000 C CNN
-F 2 "Pin_Headers:Pin_Header_Angled_1x06_Pitch2.54mm" H 700 900 50  0001 C CNN
+F 1 "IN" V 800 900 50  0000 C CNN
+F 2 "Pin_Headers:Pin_Header_Straight_1x06_Pitch2.54mm" H 700 900 50  0001 C CNN
 F 3 "" H 700 900 50  0001 C CNN
 	1    700  900
@@
 	2300 1350 2300 750
 Connection ~ 2300 750
+$Comp
+L GND #PWR07
+U 1 1 5973A1D3
+P 3500 1900
+F 0 "#PWR07" H 3500 1650 50  0001 C CNN
+F 1 "GND" H 3500 1750 50  0000 C CNN
+F 2 "" H 3500 1900 50  0001 C CNN
+F 3 "" H 3500 1900 50  0001 C CNN
+	1    3500 1900
+	1    0    0    -1
+$EndComp
+$Comp
+L VCC #PWR08
+U 1 1 5973A1E7
+P 3500 1400
+F 0 "#PWR08" H 3500 1250 50  0001 C CNN
+F 1 "VCC" H 3500 1550 50  0000 C CNN
+F 2 "" H 3500 1400 50  0001 C CNN
+F 3 "" H 3500 1400 50  0001 C CNN
+	1    3500 1400
+	1    0    0    -1
+$EndComp
+$Comp
+L CAP C13
+U 1 1 5973A488
+P 3500 1650
+F 0 "C13" V 3600 1800 50  0000 C CNN
+F 1 "100n" V 3600 1500 50  0000 C CNN
+F 2 "Capacitors_SMD:C_0805_HandSoldering" H 3500 1650 50  0001 C CNN
+F 3 "" H 3500 1650 50  0001 C CNN
+	1    3500 1650
+	1    0    0    -1
+$EndComp
 $EndSCHEMATC

Commit message: fixes
Parts:
- added R18: 100k, Resistors_SMD:R_0805_HandSoldering, symbol R
Connections:
- wire segments 23 -> 27
Changed lines of the file:
@@
 	1    0    0    -1
 $EndComp
-Wire Wire Line
-	950  1550 1500 1550
-Wire Wire Line
-	950  1650 1500 1650
-Wire Wire Line
-	950  1750 1500 1750
-Wire Wire Line
-	950  1850 1500 1850
-Wire Wire Line
-	2200 1950 2100 1950
 Text GLabel 950  1550 0    60   Input ~ 0
 ctrl_out0
@@
 Text GLabel 950  1850 0    60   Input ~ 0
 ctrl_out3
-Wire Wire Line
-	3800 2050 3800 2150
 Text GLabel 2300 1450 2    60   Input ~ 0
 ctrl_out4
@@
 Text GLabel 2300 1750 2    60   Input ~ 0
 ctrl_out7
-Wire Wire Line
-	2100 1450 2300 1450
-Wire Wire Line
-	2100 1550 2300 1550
-Wire Wire Line
-	2100 1650 2300 1650
-Wire Wire Line
-	2100 1750 2300 1750
-$Comp
-L GND #PWR01
+$Comp
+L GND #PWR3
 U 1 1 590BB78A
 P 1500 1950
-F 0 "#PWR01" H 1500 1700 50  0001 C CNN
+F 0 "#PWR3" H 1500 1700 50  0001 C CNN
 F 1 "GND" H 1500 1800 50  0000 C CNN
 F 2 "" H 1500 1950 50  0001 C CNN
@@
 $EndComp
 $Comp
-L GND #PWR02
+L GND #PWR5
 U 1 1 590BB8A5
-P 2450 1150
-F 0 "#PWR02" H 2450 900 50  0001 C CNN
-F 1 "GND" H 2450 1000 50  0000 C CNN
-F 2 "" H 2450 1150 50  0001 C CNN
-F 3 "" H 2450 1150 50  0001 C CNN
-	1    2450 1150
-	1    0    0    -1
-$EndComp
-$Comp
-L VCC #PWR03
+P 2400 1150
+F 0 "#PWR5" H 2400 900 50  0001 C CNN
+F 1 "GND" H 2400 1000 50  0000 C CNN
+F 2 "" H 2400 1150 50  0001 C CNN
+F 3 "" H 2400 1150 50  0001 C CNN
+	1    2400 1150
+	1    0    0    -1
+$EndComp
+$Comp
+L VCC #PWR6
 U 1 1 590BB9CE
 P 2450 650
-F 0 "#PWR03" H 2450 500 50  0001 C CNN
+F 0 "#PWR6" H 2450 500 50  0001 C CNN
 F 1 "VCC" H 2450 800 50  0000 C CNN
 F 2 "" H 2450 650 50  0001 C CNN
@@
 $EndComp
 $Comp
-L VCC #PWR04
+L VCC #PWR4
 U 1 1 590BB9E6
 P 2100 1250
-F 0 "#PWR04" H 2100 1100 50  0001 C CNN
+F 0 "#PWR4" H 2100 1100 50  0001 C CNN
 F 1 "VCC" H 2100 1400 50  0000 C CNN
 F 2 "" H 2100 1250 50  0001 C CNN
@@
 	0    1    1    0
 $EndComp
-Wire Wire Line
-	900  1050 2450 1050
-Wire Wire Line
-	1200 1050 1200 1450
-Wire Wire Line
-	1200 1450 1500 1450
-Wire Wire Line
-	1500 1250 1500 850
-Wire Wire Line
-	900  850  2450 850
-Wire Wire Line
-	900  750  2450 750
 $Comp
 L CONN_01X06 J1
@@
 $EndComp
 $Comp
-L GND #PWR05
+L GND #PWR2
 U 1 1 590BBE93
 P 900 1150
-F 0 "#PWR05" H 900 900 50  0001 C CNN
+F 0 "#PWR2" H 900 900 50  0001 C CNN
 F 1 "GND" H 900 1000 50  0000 C CNN
 F 2 "" H 900 1150 50  0001 C CNN
@@
 $EndComp
 $Comp
-L VCC #PWR06
+L VCC #PWR1
 U 1 1 590BBEBB
 P 900 650
-F 0 "#PWR06" H 900 500 50  0001 C CNN
+F 0 "#PWR1" H 900 500 50  0001 C CNN
 F 1 "VCC" H 900 800 50  0000 C CNN
 F 2 "" H 900 650 50  0001 C CNN
@@
 	0    1    1    0
 $EndComp
-Connection ~ 1200 1050
-Wire Wire Line
-	900  950  1350 950
-Wire Wire Line
-	1350 950  1350 1350
-Wire Wire Line
-	1350 1350 1500 1350
-Wire Wire Line
-	2200 1950 2200 950
-Wire Wire Line
-	2200 950  2450 950
-Connection ~ 1500 850
-Wire Wire Line
-	2100 1350 2300 1350
-Wire Wire Line
-	2300 1350 2300 750
-Connection ~ 2300 750
-$Comp
-L GND #PWR07
+$Comp
+L GND #PWR9
 U 1 1 5973A1D3
 P 3500 1900
-F 0 "#PWR07" H 3500 1650 50  0001 C CNN
+F 0 "#PWR9" H 3500 1650 50  0001 C CNN
 F 1 "GND" H 3500 1750 50  0000 C CNN
 F 2 "" H 3500 1900 50  0001 C CNN
@@
 $EndComp
 $Comp
-L VCC #PWR08
+L VCC #PWR8
 U 1 1 5973A1E7
 P 3500 1400
-F 0 "#PWR08" H 3500 1250 50  0001 C CNN
+F 0 "#PWR8" H 3500 1250 50  0001 C CNN
 F 1 "VCC" H 3500 1550 50  0000 C CNN
 F 2 "" H 3500 1400 50  0001 C CNN
@@
 	1    0    0    -1
 $EndComp
+$Comp
+L R R18
+U 1 1 597F86ED
+P 2950 850
+F 0 "R18" V 3030 850 50  0000 C CNN
+F 1 "100k" V 2950 850 50  0000 C CNN
+F 2 "Resistors_SMD:R_0805_HandSoldering" V 2880 850 50  0001 C CNN
+F 3 "" H 2950 850 50  0001 C CNN
+	1    2950 850
+	1    0    0    -1
+$EndComp
+Wire Wire Line
+	950  1550 1500 1550
+Wire Wire Line
+	950  1650 1500 1650
+Wire Wire Line
+	950  1750 1500 1750
+Wire Wire Line
+	950  1850 1500 1850
+Wire Wire Line
+	2200 1950 2100 1950
+Wire Wire Line
+	3800 2050 3800 2150
+Wire Wire Line
+	2100 1450 2300 1450
+Wire Wire Line
+	2100 1550 2300 1550
+Wire Wire Line
+	2100 1650 2300 1650
+Wire Wire Line
+	2100 1750 2300 1750
+Wire Wire Line
+	900  1050 2450 1050
+Wire Wire Line
+	1200 1050 1200 1450
+Wire Wire Line
+	1200 1450 1500 1450
+Wire Wire Line
+	1500 1250 1500 850
+Wire Wire Line
+	900  850  2450 850
+Wire Wire Line
+	900  750  2450 750
+Connection ~ 1200 1050
+Wire Wire Line
+	900  950  1350 950
+Wire Wire Line
+	1350 950  1350 1350
+Wire Wire Line
+	1350 1350 1500 1350
+Wire Wire Line
+	2200 1950 2200 950
+Wire Wire Line
+	2200 950  2450 950
+Connection ~ 1500 850
+Wire Wire Line
+	2100 1350 2300 1350
+Wire Wire Line
+	2300 1350 2300 750
+Connection ~ 2300 750
+Wire Wire Line
+	2950 700  2000 700
+Wire Wire Line
+	2000 700  2000 750
+Connection ~ 2000 750
+Wire Wire Line
+	2400 1150 2450 1150
+$Comp
+L GND #PWR7
+U 1 1 597F8A61
+P 2950 1100
+F 0 "#PWR7" H 2950 850 50  0001 C CNN
+F 1 "GND" H 2950 950 50  0000 C CNN
+F 2 "" H 2950 1100 50  0001 C CNN
+F 3 "" H 2950 1100 50  0001 C CNN
+	1    2950 1100
+	1    0    0    -1
+$EndComp
+Wire Wire Line
+	2950 1100 2950 1000
 $EndSCHEMATC
