File: powermgr/board/powermgmt.kicad_pcb (KiCad board)
At the start: 2 copper layers, 83.8 x 40.1 mm, 60 parts, among them IC1 CD4094, IC2 AP24x1, IC3 AP24x1, IC4 AP24x1, IC5 AP24x1, IC6 AP24x1, IC7 AP24x1, IC8 AP24x1, IC9 AP24x1, J1 IN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

Commit message: reorganize
Parts:
- moved R18 39.4 mm to (77.5, 46.1), turned to 0 degrees
Routing:
- net GND: track 866.6 -> 870.5 mm
- net Net-(IC1-Pad15): track 43.9 -> 43.0 mm
Changed lines of the file:
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@@
     (thickness 1.6)
     (drawings 70)
-    (tracks 1029)
+    (tracks 1035)
     (zones 0)
     (modules 60)
@@
   )
   (module Resistors_SMD:R_0805_HandSoldering (layer F.Cu)
-    (at 38.122 44.555 180)
+    (at 77.492 46.079)
     (descr "Resistor SMD 0805, hand soldering")
     (tags "resistor 0805")
     (attr smd)
-    (fp_text reference R18 (at 0 -1.7 180) (layer F.SilkS)
+    (fp_text reference R18 (at 0.381 4.826) (layer F.SilkS)
       (effects (font (size 1 1) (thickness 0.15)))
     )
-    (fp_text value 100k (at 0 1.75 180) (layer F.Fab)
+    (fp_text value 100k (at 0 1.75) (layer F.Fab)
       (effects (font (size 1 1) (thickness 0.15)))
     )
-    (fp_text user %R (at 0 0 180) (layer F.Fab)
+    (fp_text user %R (at 0 0) (layer F.Fab)
       (effects (font (size 0.5 0.5) (thickness 0.075)))
     )
@@
     (fp_line (start 2.35 0.9) (end 2.35 -0.9) (layer F.CrtYd) (width 0.05))
     (fp_line (start 2.35 0.9) (end -2.35 0.9) (layer F.CrtYd) (width 0.05))
-    (pad 1 smd rect (at -1.35 0 180) (size 1.5 1.3) (layers F.Cu F.Paste F.Mask)
+    (pad 1 smd rect (at -1.35 0) (size 1.5 1.3) (layers F.Cu F.Paste F.Mask)
       (net 6 "Net-(IC1-Pad15)"))
-    (pad 2 smd rect (at 1.35 0 180) (size 1.5 1.3) (layers F.Cu F.Paste F.Mask)
+    (pad 2 smd rect (at 1.35 0) (size 1.5 1.3) (layers F.Cu F.Paste F.Mask)
       (net 26 GND))
     (model ${KISYS3DMOD}/Resistors_SMD.3dshapes/R_0805.wrl
@@
   (segment (start 70.739 48.768) (end 70.739 48.5775) (width 0.25) (layer F.Cu) (net 4))
   (segment (start 55.978 40.143) (end 55.978 40.034) (width 0.25) (layer F.Cu) (net 4))
-  (segment (start 39.472 44.555) (end 40.662 44.555) (width 0.25) (layer F.Cu) (net 6) (status 400000))
-  (segment (start 40.662 44.555) (end 42.44 46.333) (width 0.25) (layer F.Cu) (net 6))
+  (segment (start 76.142 46.079) (end 76.142 48.445) (width 0.25) (layer F.Cu) (net 6))
+  (segment (start 76.142 48.445) (end 75.819 48.768) (width 0.25) (layer F.Cu) (net 6))
   (segment (start 75.819 48.768) (end 75.819 48.514) (width 0.25) (layer F.Cu) (net 6))
   (segment (start 75.819 48.514) (end 71.0565 43.7515) (width 0.25) (layer F.Cu) (net 6))
@@
   (segment (start 76.708 28.288) (end 76.708 22.831) (width 1) (layer F.Cu) (net 25))
   (segment (start 76.708 22.831) (end 75.826 21.949) (width 1) (layer F.Cu) (net 25))
-  (segment (start 33.528 48.725) (end 33.698 48.725) (width 0.5) (layer F.Cu) (net 26) (status C00000))
-  (segment (start 33.698 48.725) (end 36.772 45.651) (width 0.5) (layer F.Cu) (net 26) (status 400000))
-  (segment (start 36.772 45.651) (end 36.772 44.555) (width 0.5) (layer F.Cu) (net 26) (status 800000))
+  (segment (start 78.842 46.079) (end 79.016 46.079) (width 0.25) (layer F.Cu) (net 26))
+  (segment (start 79.016 46.079) (end 81.662 48.725) (width 0.25) (layer F.Cu) (net 26))
+  (segment (start 81.662 48.725) (end 82.042 48.725) (width 0.25) (layer F.Cu) (net 26))
+  (segment (start 65.326 21.949) (end 65.326 17.971) (width 1.75) (layer F.Cu) (net 26))
+  (segment (start 51.326 21.949) (end 51.326 17.521) (width 1.75) (layer F.Cu) (net 26))
+  (segment (start 51.076 17.758) (end 51.076 17.521) (width 1.75) (layer F.Cu) (net 26))
+  (segment (start 51.089 17.758) (end 51.076 17.758) (width 1.75) (layer F.Cu) (net 26))
+  (segment (start 51.326 17.521) (end 51.089 17.758) (width 1.75) (layer F.Cu) (net 26))
+  (segment (start 33.528 48.725) (end 33.698 48.725) (width 0.5) (layer F.Cu) (net 26))
   (segment (start 27.456 28.021) (end 27.456 24.819) (width 1.75) (layer F.Cu) (net 26))
   (segment (start 27.456 24.819) (end 30.326 21.949) (width 1.75) (layer F.Cu) (net 26))
@@
   (segment (start 72.456 17.641) (end 72.456 17.521) (width 2) (layer B.Cu) (net 26))
   (segment (start 72.326 17.771) (end 72.456 17.641) (width 2) (layer B.Cu) (net 26))
-  (segment (start 65.326 21.949) (end 65.326 17.971) (width 2) (layer B.Cu) (net 26))
   (segment (start 65.326 17.971) (end 65.278 17.923) (width 2) (layer B.Cu) (net 26))
   (segment (start 58.326 21.949) (end 58.326 18.591) (width 2) (layer B.Cu) (net 26))
@@
   (segment (start 30.326 19.151) (end 31.956 17.521) (width 3) (layer F.Cu) (net 26))
   (segment (start 58.456 17.521) (end 79.206 17.521) (width 3) (layer F.Cu) (net 26))
-  (segment (start 44.206 17.521) (end 58.456 17.521) (width 3) (layer F.Cu) (net 26))
+  (segment (start 44.206 17.521) (end 51.076 17.521) (width 3) (layer F.Cu) (net 26))
+  (segment (start 51.076 17.521) (end 58.456 17.521) (width 3) (layer F.Cu) (net 26))
   (segment (start 37.456 17.521) (end 44.206 17.521) (width 3) (layer F.Cu) (net 26))
   (segment (start 79.798 26.013) (end 79.798 22.421) (width 1.5) (layer F.Cu) (net 26))
