File: powerleaf/powerleaf.kicad_pcb (KiCad board)
At the start: 2 copper layers, 8.9 x 49.5 mm, 20 parts, among them J1 Conn_01x02, J2 Cap, J3 Conn_01x03, U1 MCP16252-I_CH, U2 MCP1711

Commit message: stuff
Parts:
- added C10: 10uF, Capacitor_SMD:C_0805_2012Metric_Pad1.18x1.45mm_HandSolder, B.Cu at (16.2, 27.2)
- added C8: 100n, Capacitor_SMD:C_0805_2012Metric_Pad1.18x1.45mm_HandSolder, F.Cu at (17.1, 52.5)
- added C9: 10uF, Capacitor_SMD:C_0805_2012Metric_Pad1.18x1.45mm_HandSolder, B.Cu at (16.2, 29.4)
- added E1: SPARK_GAP, 0_eurocad:SparkGap-0.3mm, F.Cu at (17.5, 61.5)
- moved F1 0.18 mm to (13.3, 57.1)
- moved R3 0.07 mm to (12.9, 22.6)
Connections:
- D1 pad 2: Net-(D1-Pad2) -> Vin
- F1 pad 1: Net-(D1-Pad2) -> Vin
- F1 pad 2: Vin -> Net-(E1-Pad1)
- J1 pad 1: Vin -> Net-(E1-Pad1)
Routing:
- net GND: track 78.4 -> 95.7 mm, vias 19 -> 20
- net Vin: track 43.6 -> 36.7 mm
- net Vcap: track 33.0 -> 39.2 mm
- net /Vsw: track 30.8 -> 36.9 mm, vias 0 -> 2
- net Net-(E1-Pad1): track 0.00 -> 5.18 mm
- net Net-(L1-Pad2): track 0.00 -> 3.44 mm
- net Net-(D1-Pad2): track 2.40 -> 0.00 mm
