File: rootcore/rootcore/rootcore.kicad_pcb (KiCad board)
At the start: 2 copper layers, 20 parts, among them J1 Conn_02x20_Odd_Even, J2 Conn_02x20_Odd_Even, J3 Conn_02x08_Odd_Even, J4 Conn_01x04_Male, U1 STM32F373VCTx, U2 LM13700, U3 AP1117-15, U4 LM4040DCK-2.5, Y1 Crystal

Commit message: micro routed
Parts:
- added C6: 10n, Capacitor_SMD:C_0805_2012Metric_Pad1.18x1.45mm_HandSolder, F.Cu at (25.7, 54.2)
- added C7: 10n, Capacitor_SMD:C_0805_2012Metric_Pad1.18x1.45mm_HandSolder, F.Cu at (37.8, 51.2)
- added J5: Conn_01x02_Male, Connector_PinHeader_2.54mm:PinHeader_1x02_P2.54mm_Vertical, F.Cu at (34.4, 47.2)
- U1: value STM32F373VCTx -> STM32F373RCTx; footprint Package_QFP:LQFP-100_14x14mm_P0.5mm -> Package_QFP:LQFP-64_10x10mm_P0.5mm
- moved C5 2.73 mm to (34.7, 70.7)
- moved U1 0.39 mm to (35.3, 61.2)
Connections:
- J1 pad 10: (no net) -> PC11
- J1 pad 11: (no net) -> PB4
- J1 pad 12: (no net) -> PA15
- J1 pad 13: (no net) -> PB6
- J1 pad 14: (no net) -> PB5
- J1 pad 15: (no net) -> PF7
- J1 pad 16: (no net) -> PB7
- J1 pad 17: (no net) -> PA12
- J1 pad 18: (no net) -> PF6
- J1 pad 19: (no net) -> PA10
- J1 pad 20: (no net) -> PA11
- J1 pad 21: (no net) -> PA8
- J1 pad 22: (no net) -> PA9
- J1 pad 23: (no net) -> PC8
- J1 pad 24: (no net) -> PC9
- J1 pad 25: (no net) -> PC6
- J1 pad 26: (no net) -> PC7
- J1 pad 27: (no net) -> PB15
- J1 pad 28: (no net) -> PD8
- J1 pad 29: (no net) -> GND
- J1 pad 30: (no net) -> PB14
- J1 pad 4: (no net) -> PB9
- J1 pad 5: (no net) -> PB3
- J1 pad 6: (no net) -> PB8
- J1 pad 7: (no net) -> PC12
- J1 pad 8: (no net) -> PD2
- J1 pad 9: (no net) -> PC10
- J2 pad 10: PA5 -> PC2
- J2 pad 11: PA6 -> PC3
- J2 pad 12: PA7 -> PA0
- J2 pad 13: PC4 -> PA1
- J2 pad 14: PC5 -> PA2
- J2 pad 15: PB0 -> PA3
- J2 pad 16: PB1 -> PA4
- J2 pad 17: PB2 -> PA5
- J2 pad 18: PE7 -> PA6
- J2 pad 19: PE8 -> PA7
- J2 pad 20: PE9 -> PC4
- J2 pad 21: PE10 -> PC5
- J2 pad 22: PE11 -> PB0
- J2 pad 23: PE12 -> PB1
- J2 pad 24: PE13 -> PB2
- J2 pad 25: PE14 -> PE8
- J2 pad 26: PE15 -> PE9
- J2 pad 27: PB10 -> GND
- J2 pad 28: (no net) -> GND
- J2 pad 4: PA1 -> Ref2v5
- J2 pad 5: PA2 -> PC13
- J2 pad 6: PA0 -> PC14
- J2 pad 7: PA3 -> PC15
- J2 pad 8: PF4 -> PC0
- J2 pad 9: PA4 -> PC1
- U1 pad 1: (no net) -> 3v3
- U1 pad 10: (no net) -> PC2
- U1 pad 11: (no net) -> PC3
- U1 pad 12: PF0 -> GNDA
- U1 pad 13: PF1 -> 3v3a
- U1 pad 14: (no net) -> PA0
- U1 pad 15: (no net) -> PA1
- U1 pad 16: (no net) -> PA2
- U1 pad 17: (no net) -> Ref2v5
- U1 pad 18: (no net) -> PA3
- U1 pad 19: (no net) -> 3v3
- U1 pad 2: (no net) -> PC13
- U1 pad 20: GNDA -> PA4
- U1 pad 21: 3v3a -> PA5
- U1 pad 22: Ref2v5 -> PA6
- U1 pad 23: PA0 -> PA7
- U1 pad 24: PA1 -> PC4
- U1 pad 25: PA2 -> PC5
- U1 pad 26: PA3 -> PB0
- U1 pad 27: PF4 -> PB1
- U1 pad 28: 3v3 -> PB2
- U1 pad 29: PA4 -> PE8
- U1 pad 3: (no net) -> PC14
- U1 pad 30: PA5 -> PE9
- U1 pad 31: PA6 -> GNDA
- U1 pad 32: PA7 -> 3v3a
- U1 pad 33: PC4 -> Ref2v5
- U1 pad 34: PC5 -> PB14
- U1 pad 35: PB0 -> PB15
- U1 pad 36: PB1 -> PD8
- U1 pad 37: PB2 -> PC6
- U1 pad 38: PE7 -> PC7
- U1 pad 39: PE8 -> PC8
- U1 pad 4: (no net) -> PC15
- U1 pad 40: PE9 -> PC9
- U1 pad 41: PE10 -> PA8
- U1 pad 42: PE11 -> PA9
- U1 pad 43: PE12 -> PA10
- U1 pad 44: PE13 -> PA11
- U1 pad 45: PE14 -> PA12
- U1 pad 46: PE15 -> PA13
- U1 pad 47: PB10 -> PF6
- U1 pad 48: GNDA -> PF7
- U1 pad 49: GNDA -> PA14
- U1 pad 5: (no net) -> PF0
- U1 pad 50: 3v3a -> PA15
- U1 pad 51: 3v3a -> PC10
- U1 pad 52: Ref2v5 -> PC11
- U1 pad 53: (no net) -> PC12
- U1 pad 54: (no net) -> PD2
- U1 pad 55: (no net) -> PB3
- U1 pad 56: (no net) -> PB4
- U1 pad 57: (no net) -> PB5
- U1 pad 58: (no net) -> PB6
- U1 pad 59: (no net) -> PB7
- U1 pad 6: 3v3 -> PF1
- U1 pad 60: (no net) -> BOOT0
- U1 pad 61: (no net) -> PB8
- U1 pad 62: (no net) -> PB9
- U1 pad 63: (no net) -> GND
- U1 pad 64: (no net) -> 3v3
- U1 pad 7: (no net) -> NRST
- U1 pad 8: (no net) -> PC0
- U1 pad 9: (no net) -> PC1
Routing:
- net GND: track 121.8 -> 192.1 mm, vias 0 -> 6
- net PB7: track 0.00 -> 55.5 mm, vias 0 -> 1
- net PB14: track 0.00 -> 54.3 mm
- net PD8: track 0.00 -> 52.2 mm
- net PB5: track 0.00 -> 50.6 mm, vias 0 -> 1
- net PB15: track 0.00 -> 50.4 mm
- net PC7: track 0.00 -> 50.1 mm
- net PB6: track 0.00 -> 49.7 mm, vias 0 -> 1
- net PB10: track 49.1 -> 0.00 mm, vias 1 -> 0
- net PE15: track 48.7 -> 0.00 mm
- net PC6: track 0.00 -> 48.3 mm
- net PC9: track 0.00 -> 47.8 mm
- net PE14: track 47.2 -> 0.00 mm, vias 1 -> 0
- net PE13: track 46.5 -> 0.00 mm
- net PC3: track 0.00 -> 46.3 mm
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- added copper zone on B.Cu, net GND
- added copper zone on F.Cu, net GNDA

Commit message: base layoyut done
Parts:
- added C10: 2.2u, Capacitor_SMD:C_0805_2012Metric_Pad1.18x1.45mm_HandSolder, F.Cu at (28.8, 115.2)
- added C11: 2.2u, Capacitor_SMD:C_0805_2012Metric_Pad1.18x1.45mm_HandSolder, F.Cu at (28.6, 111.8)
- added C12: 100n, Capacitor_SMD:C_0805_2012Metric_Pad1.18x1.45mm_HandSolder, F.Cu at (36.8, 108.5)
- added C13: 100n, Capacitor_SMD:C_0805_2012Metric_Pad1.18x1.45mm_HandSolder, F.Cu at (41.2, 114.7)
- added C14: 100n, Capacitor_SMD:C_0805_2012Metric_Pad1.18x1.45mm_HandSolder, F.Cu at (28.9, 125.0)
- added C15: 100n, Capacitor_SMD:C_0805_2012Metric_Pad1.18x1.45mm_HandSolder, F.Cu at (42.5, 119.0)
- added C16: 10u, Capacitor_SMD:C_0805_2012Metric_Pad1.18x1.45mm_HandSolder, F.Cu at (22.5, 38.8)
- added C17: 10u, Capacitor_SMD:C_0805_2012Metric_Pad1.18x1.45mm_HandSolder, F.Cu at (23.0, 35.8)
- added C18: 10u, Capacitor_SMD:C_0805_2012Metric_Pad1.18x1.45mm_HandSolder, F.Cu at (22.5, 41.1)
- added C19: 10u, Capacitor_SMD:C_0805_2012Metric_Pad1.18x1.45mm_HandSolder, F.Cu at (44.5, 36.5)
- added C8: 100n, Capacitor_SMD:C_0805_2012Metric_Pad1.18x1.45mm_HandSolder, F.Cu at (29.0, 118.1)
- added C9: 100n, Capacitor_SMD:C_0805_2012Metric_Pad1.18x1.45mm_HandSolder, F.Cu at (32.4, 108.5)
- added R3: 20k, Resistor_SMD:R_0805_2012Metric_Pad1.20x1.40mm_HandSolder, F.Cu at (27.9, 128.0)
- added R4: 13k, Resistor_SMD:R_0805_2012Metric_Pad1.20x1.40mm_HandSolder, F.Cu at (29.9, 128.0)
- added R5: 1k, Resistor_SMD:R_0805_2012Metric_Pad1.20x1.40mm_HandSolder, F.Cu at (32.9, 129.7)
- added R6: 20k, Resistor_SMD:R_0805_2012Metric_Pad1.20x1.40mm_HandSolder, F.Cu at (27.8, 122.0)
- added R7: 13k, Resistor_SMD:R_0805_2012Metric_Pad1.20x1.40mm_HandSolder, F.Cu at (29.9, 122.0)
- added R8: 1k, Resistor_SMD:R_0805_2012Metric_Pad1.20x1.40mm_HandSolder, F.Cu at (36.7, 129.7)
- added R9: 0, NetTie:NetTie-2_SMD_Pad0.5mm, F.Cu at (31.1, 119.0)
- added U5: PCM5100, Package_SO:TSSOP-20_4.4x6.5mm_P0.65mm, F.Cu at (34.9, 113.6)
- U2: value LM13700 -> TL074; footprint Package_SO:SOIC-16_3.9x9.9mm_P1.27mm -> Package_SO:SOIC-14_3.9x8.7mm_P1.27mm
- moved U2 3.07 mm to (34.9, 124.1)
Connections:
- net PA10 renamed DAC_DIN
- net PA11 renamed DAC_LRCK
- net PA8 renamed DAC_BCK
- J1 pad 31: (no net) -> 3v3
- J1 pad 32: (no net) -> -12v
- J1 pad 33: (no net) -> OP1_OUT
- J1 pad 34: (no net) -> OP1_INN
- J1 pad 35: (no net) -> OP1_INP
- J1 pad 36: (no net) -> OP2_INP
- J1 pad 37: (no net) -> OP2_INN
- J1 pad 38: (no net) -> OP2_OUT
- J2 pad 29: (no net) -> 12v
- J2 pad 30: (no net) -> GND
- J2 pad 31: (no net) -> 12v
- J2 pad 32: (no net) -> GND
- J2 pad 33: (no net) -> 12v
- J2 pad 34: (no net) -> GND
- J2 pad 35: (no net) -> 12v
- J2 pad 36: (no net) -> GND
- J2 pad 37: (no net) -> OUT_R
- J2 pad 38: (no net) -> OUT_L
- U2 pad 1: (no net) -> Net-(R7-Pad2)
- U2 pad 10: (no net) -> OP2_INP
- U2 pad 11: (no net) -> -12v
- U2 pad 12: (no net) -> OP1_INP
- U2 pad 13: (no net) -> OP1_INN
- U2 pad 14: (no net) -> OP1_OUT
- U2 pad 2: (no net) -> DAC_R
- U2 pad 3: (no net) -> Net-(R6-Pad1)
- U2 pad 4: (no net) -> 12v
- U2 pad 5: (no net) -> Net-(R3-Pad1)
- U2 pad 6: (no net) -> DAC_L
- U2 pad 7: (no net) -> Net-(R4-Pad2)
- U2 pad 8: (no net) -> OP2_OUT
- U2 pad 9: (no net) -> OP2_INN
Routing:
- net -12v: track 70.9 -> 181.3 mm, vias 0 -> 4
- net 3v3: track 99.2 -> 197.4 mm, vias 5 -> 8
- net GND: track 192.1 -> 284.6 mm, vias 6 -> 16
- net 12v: track 70.9 -> 130.6 mm, vias 0 -> 3
- net GNDS: track 0.00 -> 19.9 mm
- net OUT_R: track 0.00 -> 19.0 mm, vias 0 -> 1
- net DAC_L: track 0.00 -> 16.9 mm, vias 0 -> 2
- net DAC_DIN: track 41.9 -> 58.3 mm, vias 0 -> 2
- net DAC_LRCK: track 43.7 -> 59.9 mm, vias 0 -> 2
- net DAC_BCK: track 44.0 -> 59.2 mm, vias 0 -> 2
- net Net-(R7-Pad2): track 0.00 -> 14.8 mm
- net OP1_INN: track 0.00 -> 11.5 mm
- net OP2_INP: track 0.00 -> 11.4 mm
- net OP2_OUT: track 0.00 -> 11.4 mm
- net DAC_R: track 0.00 -> 9.97 mm, vias 0 -> 2
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- added copper zone on F.Cu, net GNDS
Other:
- board outline added: 30.2 x 105.5 mm

Commit message: stuff
Parts:
- added C20: 22u, Capacitor_SMD:C_0805_2012Metric_Pad1.18x1.45mm_HandSolder, F.Cu at (22.4, 44.2)
- added C21: 22u, Capacitor_SMD:C_0805_2012Metric_Pad1.18x1.45mm_HandSolder, F.Cu at (25.5, 42.1)
- added C22: 100n, Capacitor_SMD:C_0805_2012Metric_Pad1.18x1.45mm_HandSolder, F.Cu at (33.3, 37.3)
- added C23: 22u, Capacitor_SMD:C_0805_2012Metric_Pad1.18x1.45mm_HandSolder, F.Cu at (35.4, 37.3)
- added C24: 22u, Capacitor_SMD:C_0805_2012Metric_Pad1.18x1.45mm_HandSolder, F.Cu at (37.5, 37.3)
- added C25: 100n, Capacitor_SMD:C_0805_2012Metric_Pad1.18x1.45mm_HandSolder, F.Cu at (40.2, 125.0)
- added C26: 22u, Capacitor_SMD:C_0805_2012Metric_Pad1.18x1.45mm_HandSolder, F.Cu at (42.4, 125.0)
- added D1: LED, LED_SMD:LED_0805_2012Metric, F.Cu at (32.1, 52.3)
- added L2: 100u >300mA, 0_eurocad:YP0302, F.Cu at (24.9, 36.9)
- added L3: 100u >300mA, 0_eurocad:YP0302, F.Cu at (47.9, 34.0)
- added L4: 100u >300mA, 0_eurocad:YP0302, F.Cu at (29.8, 36.9)
- added R10: 220, Resistor_SMD:R_0805_2012Metric_Pad1.20x1.40mm_HandSolder, F.Cu at (28.3, 50.8)
- C16, C17, C18, C19: value 10u -> 22u
- C6: value 10n -> 100n
- C7: value 10n -> 22u
- U4: value LM4040DCK-2.5 -> LM4040DBZ-2.5; footprint Package_TO_SOT_SMD:SOT-353_SC-70-5 -> Package_TO_SOT_SMD:SOT-23
- Y1: value Crystal -> Crystal_GND24; footprint Crystal:Crystal_SMD_7050-2Pin_7.0x5.0mm -> Crystal:Crystal_SMD_TXC_7M-4Pin_3.2x2.5mm_HandSoldering
- moved C17 10.6 mm to (23.7, 46.4), turned to 0 degrees
- moved C16 7.11 mm to (22.6, 31.7), turned to 270 degrees
- moved C1 6.29 mm to (35.8, 42.1), turned to 270 degrees
- moved C2 5.45 mm to (27.7, 42.1)
- moved C19 1.52 mm to (43.3, 35.5), turned to 180 degrees
- moved U3 1.35 mm to (43.0, 41.6)
- moved C18 1.02 mm to (22.4, 42.2)
- moved Y1 0.82 mm to (31.7, 41.7)
- moved U4 0.57 mm to (23.1, 57.9), turned to 0 degrees
- moved C6 0.46 mm to (26.1, 53.9)
Connections:
- J1 pad 39: (no net) -> GND
- J1 pad 40: (no net) -> GND
- J2 pad 39: (no net) -> GND
- J2 pad 40: (no net) -> GND
- J3 pad 15: -12v -> -12vRAW
- J3 pad 16: -12v -> -12vRAW
- J3 pad 5: 5v -> 5vRAW
- J3 pad 6: 5v -> 5vRAW
- J3 pad 7: 12v -> 12vRAW
- J3 pad 8: 12v -> 12vRAW
- U4 pad 1: GNDA -> Ref2v5
- U4 pad 2: (no net) -> GNDA
- U4 pad 3: Ref2v5 -> (no net)
- U5 pad 11: GND -> 3v3
- Y1 pad 2: PF1 -> GND
Routing:
- net GND: track 284.6 -> 545.3 mm, vias 16 -> 57
- net GNDA: track 41.3 -> 65.2 mm
- net 12vRAW: track 0.00 -> 21.5 mm, vias 0 -> 1
- net -12vRAW: track 0.00 -> 6.73 mm
- net 5vRAW: track 0.00 -> 6.29 mm
- net 3v3: track 197.4 -> 203.4 mm, vias 8 -> 25
- net 5v: track 69.9 -> 64.0 mm
- net PB7: track 55.5 -> 49.7 mm
- net PB6: track 50.2 -> 45.2 mm
- net PC13: track 41.6 -> 45.5 mm, vias 1 -> 0
- net PB5: track 50.8 -> 47.0 mm
- net Ref2v5: track 51.6 -> 55.0 mm, vias 4 -> 3
- net 12v: track 130.6 -> 133.7 mm, vias 3 -> 6
- net -12v: track 181.3 -> 184.3 mm, vias 4 -> 5
- net PF1: track 22.9 -> 20.0 mm
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- added copper zone on B.Cu, net 3v3
- added copper zone on F.Cu, net 3v3
- removed copper zone on F.Cu, net GNDA
Other:
- board text added: "(DAC!)"
- board text added: "+"
- board text added: "+5v"
- board text added: "-"
- board text added: "-12V|GND"
- board text added: "-12v|3.3v"
- board text added: "2.5v ref|12V"
- board text added: "3v3"
- board text added: "3v3|GND"
- board text added: "B"
- board text added: "BOOT"
- board text added: "CLK"
- board text added: "DIO"
- board text added: "GND"
- board text added: "GND|12v"
- board text added: "GND|GND"
- board text added: "JLCJLCJLCJLC"
- board text added: "OP1_IN+|OP2_IN+"
- board text added: "OP1_IN-|OP1_OUT"
- board text added: "OP2_OUT|OP2_IN-"
- board text added: "OUT_L|OUT_R"
- board text added: "PA0|PC3"
- board text added: "PA11|PA10"
- board text added: "PA2|PA1"
- board text added: "PA4|PA3"
- board text added: "PA6|PA5"
- board text added: "PA9|PA8"
- board text added: "PB0|PB0"
- board text added: "PB0|PC5"
- board text added: "PB14|GND"
- board text added: "PB2|PB1"
- board text added: "PB5|PB6"
- board text added: "PB7|PF7"
- board text added: "PB8|PB3"
- board text added: "PB9|5v"
- board text added: "PC0|PC15"
- board text added: "PC11|PC10"
- board text added: "PC14|PC13"
- board text added: "PC2|PC1"
- board text added: "PC4|PA7"
- board text added: "PC7|PC6"
- board text added: "PC9|PC8"
- board text added: "PD8|PB15"
- board text added: "PE9|PE8"
- board text added: "PF6|PA12"
- board text added: "ROOTCORE"
- board text added: "RST"
- board text added: "⏚"
