File: rootcore/rootcore/rootcore.sch (KiCad schematic (older format))
At the start: 17 parts, among them J1 Conn_02x20_Odd_Even, J2 Conn_02x20_Odd_Even, J3 Conn_02x08_Odd_Even, J4 Conn_01x04_Male, U1 STM32F373VCTx, U2 LM13700, U3 AP1117-15, U4 LM4040DCK-2.5, Y1 Crystal

Commit message: micro routed
Parts:
- removed U1: STM32F373VCTx, Package_QFP:LQFP-100_14x14mm_P0.5mm, symbol MCU_ST_STM32F3:STM32F373VCTx
- added C6, C7: 10n, Capacitor_SMD:C_0805_2012Metric_Pad1.18x1.45mm_HandSolder, symbol Device:C
- added J5: Conn_01x02_Male, Connector_PinHeader_2.54mm:PinHeader_1x02_P2.54mm_Vertical, symbol Connector:Conn_01x02_Male
- added U1: STM32F373RCTx, Package_QFP:LQFP-64_10x10mm_P0.5mm, symbol MCU_ST_STM32F3:STM32F373RCTx
Connections:
- net labels added: BOOT0, NRST, PF7
- net labels removed: PB10, PD0, PD1, PD10, PD11, PD12, PD13, PD14, PD15, PD3, PD4, PD5, PD6, PD7, PD9, PE0, PE1, PE10, PE11, PE12, PE13, PE14, PE15, PE2, PE3, PE4, PE5, PE6, PE7, PF10, PF2, PF4, PF9
- wire segments 151 -> 77

Commit message: base layoyut done
Parts:
- removed U2: LM13700, Package_SO:SOIC-16_3.9x9.9mm_P1.27mm, symbol Amplifier_Operational:LM13700
- added C10, C11: 2.2u, Capacitor_SMD:C_0805_2012Metric_Pad1.18x1.45mm_HandSolder, symbol Device:C
- added C12, C13, C14, C15, C8, C9: 100n, Capacitor_SMD:C_0805_2012Metric_Pad1.18x1.45mm_HandSolder, symbol Device:C
- added C16, C17, C18, C19: 10u, Capacitor_SMD:C_0805_2012Metric_Pad1.18x1.45mm_HandSolder, symbol Device:C
- added R3, R6: 20k, Resistor_SMD:R_0805_2012Metric_Pad1.20x1.40mm_HandSolder, symbol Device:R
- added R4, R7: 13k, Resistor_SMD:R_0805_2012Metric_Pad1.20x1.40mm_HandSolder, symbol Device:R
- added R5, R8: 1k, Resistor_SMD:R_0805_2012Metric_Pad1.20x1.40mm_HandSolder, symbol Device:R
- added R9: 0, NetTie:NetTie-2_SMD_Pad0.5mm, symbol Device:R
- added U2: TL074, Package_SO:SOIC-14_3.9x8.7mm_P1.27mm, symbol Amplifier_Operational:TL074
- added U5: PCM5100, Package_SO:TSSOP-20_4.4x6.5mm_P0.65mm, symbol Audio:PCM5100
Connections:
- net labels added: DAC_BCK, DAC_DIN, DAC_L, DAC_LRCK, DAC_R, GNDS, OP1_INN, OP1_INP, OP1_OUT, OP2_INN, OP2_INP, OP2_OUT, OUT_L, OUT_R
- wire segments 77 -> 137

Commit message: stuff
Parts:
- removed U4: LM4040DCK-2.5, Package_TO_SOT_SMD:SOT-353_SC-70-5, symbol Reference_Voltage:LM4040DCK-2.5
- removed Y1: Crystal, Crystal:Crystal_SMD_7050-2Pin_7.0x5.0mm, symbol Device:Crystal
- added C20, C21, C23, C24, C26: 22u, Capacitor_SMD:C_0805_2012Metric_Pad1.18x1.45mm_HandSolder, symbol Device:C
- added C22, C25: 100n, Capacitor_SMD:C_0805_2012Metric_Pad1.18x1.45mm_HandSolder, symbol Device:C
- added D1: LED, LED_SMD:LED_0805_2012Metric, symbol Device:LED
- added L2, L3, L4: 100u >300mA, 0_eurocad:YP0302, symbol Device:L
- added R10: 220, Resistor_SMD:R_0805_2012Metric_Pad1.20x1.40mm_HandSolder, symbol Device:R
- added U4: LM4040DBZ-2.5, Package_TO_SOT_SMD:SOT-23, symbol Reference_Voltage:LM4040DBZ-2.5
- added Y1: Crystal_GND24, Crystal:Crystal_SMD_TXC_7M-4Pin_3.2x2.5mm_HandSoldering, symbol Device:Crystal_GND24
- C1, C2: LCSC (none) -> C1797
- C10, C11: LCSC (none) -> C49217
- C12, C13, C14, C15, C3, C4, C5, C8, C9: LCSC (none) -> C49678; MPN (none) -> CC0805KRX7R9BB104
- C16, C17, C18, C19: value 10u -> 22u; LCSC (none) -> C45783
- C6: value 10n -> 100n; LCSC (none) -> C49678; MPN (none) -> CC0805KRX7R9BB104
- C7: value 10n -> 22u; LCSC (none) -> C45783
- L1: LCSC (none) -> C68035; MPN (none) -> SWPA5040S101MT
- R2, R5, R8: LCSC (none) -> C17513; MPN (none) -> RC0805FR-071KL
- R3, R6: LCSC (none) -> C4328; MPN (none) -> RC0805JR-0720KL
- R4, R7: LCSC (none) -> C17455; MPN (none) -> RC0805FR-0713KL
- U1: LCSC (none) -> C84174; MPN (none) -> STM32F373RCT6
- U2: LCSC (none) -> C12594; MPN (none) -> TL074IDR; jlc_offset (none) -> 270
- U2: LCSC (none) -> C12594; MPN (none) -> TL074IDR; jlc_offset (none) -> 90
- U3: LCSC (none) -> C6186; MPN (none) -> AMS1117-3.3; jlc_offset (none) -> 180
- U5: LCSC (none) -> C131154; MPN (none) -> PCM5100APWR
Connections:
- net -12v: now also C21.2, C25.2, C26.2, L3.2; no longer J3.15 (Pin_15), J3.16 (Pin_16)
- net 12v: now also C20.1, C25.1, C26.1, L2.2; no longer J3.7 (Pin_7), J3.8 (Pin_8)
- net 3v3: now also U5.11 (FLT)
- net 5v: now also U3.3 (VI), C22.1, C23.1, C24.1, L4.2; no longer J3.5 (Pin_5), J3.6 (Pin_6)
- net GND: now also J1.39 (Pin_39), J1.40 (Pin_40), J2.39 (Pin_39), J2.40 (Pin_40), C20.2, C21.1, C22.2, C23.2, C24.2, R10.2, Y1.2, Y1.4; no longer U5.11 (FLT)
- net GNDA: now also U4.2 (A)
- net PC13: now also D1.2 (A)
- net PF0: now also Y1.1
- net PF1: now also Y1.3
- net Ref2v5: now also U4.1 (K)
- new net: D1.1 (K), R10.1
- new net -12vRAW: J3.15 (Pin_15), J3.16 (Pin_16), L3.1
- new net 12vRAW: J3.7 (Pin_7), J3.8 (Pin_8), L2.1
- new net 5vRAW: J3.5 (Pin_5), J3.6 (Pin_6), L4.1
Other:
- moved on the sheet: C14, C15, C16, C17, C18, C19, U2E
